Commit message: Update etrobo_spike/model.sdf

File: urdf/etrobo_spike.urdf (robot description, URDF)
Before this commit: robot etrobo_spike, 5 links, 4 joints
Links:
- link base_link: mass 5.0 -> 1.0; geometry collision box size=0.19965 0.083846 0.135762; visual box size=0.19965 0.083846 0.135762
- link caster_back_link: mass 0.1 -> 0.01; geometry collision sphere radius=0.015972; visual sphere radius=0.015972
- link wheel_left_link: mass 0.2 -> 0.1; geometry collision cylinder length=0.015972 radius=0.028; visual cylinder length=0.015972 radius=0.028
- link wheel_right_link: mass 0.2 -> 0.1; geometry collision cylinder length=0.015972 radius=0.028; visual cylinder length=0.015972 radius=0.028
Joints:
- joint base_joint: origin xyz=0 0 0.01 rpy=0 0 0 -> xyz=0 0 0.083853 rpy=0 0 0
- joint caster_back_joint: origin xyz=0 0 0 rpy=0 0 0 -> xyz=-0.143748 0 0.015972 rpy=0 0 0
- joint wheel_left_joint: origin xyz=0 0.18 0.072 rpy=0 0 0 -> xyz=0 0.043423 0.028 rpy=0 0 0
- joint wheel_right_joint: origin xyz=0 -0.18 0.072 rpy=0 0 0 -> xyz=0 -0.043423 0.028 rpy=0 0 0

Commit message: Modify models/etrobo_spike/model.sdf

File: urdf/etrobo_spike.urdf (robot description, URDF)
Before this commit: robot etrobo_spike, 5 links, 4 joints
Links:
- removed link base_link
- added link arm_link, mass 0.031; collision box size=0.024 0.056 0.048; visual box size=0.024 0.056 0.048
- added link body_link, mass 0.434; collision box size=0.112 0.088 0.08; visual box size=0.112 0.088 0.08
- added link container_link, mass 0.354; collision box size=0.096 0.104 0.088; visual box size=0.096 0.104 0.088
- added link head_link, mass 0.124; collision box size=0.080 0.072 0.072; visual box size=0.080 0.072 0.072
- link caster_back_link: mass 0.01 -> 0.0096; geometry collision sphere radius=0.012; visual sphere radius=0.012
- link wheel_left_link: mass 0.1 -> 0.014; geometry collision cylinder length=0.008 radius=0.028; visual cylinder length=0.008 radius=0.028
- link wheel_right_link: mass 0.1 -> 0.014; geometry collision cylinder length=0.008 radius=0.028; visual cylinder length=0.008 radius=0.028
Joints:
- added joint arm_joint: type fixed, parent body_link, child arm_link, origin xyz=0 0 0 rpy=0 0 0
- added joint container_joint: type fixed, parent body_link, child container_link, origin xyz=0 0 0 rpy=0 0 0
- added joint head_joint: type fixed, parent body_link, child head_link, origin xyz=0 0 0 rpy=0 0 0
- joint base_joint: child base_link -> body_link; origin xyz=0 0 0.083853 rpy=0 0 0 -> xyz=0 0 0.028 rpy=0 0 0
- joint caster_back_joint: origin xyz=-0.143748 0 0.015972 rpy=0 0 0 -> xyz=-0.021348 0 -0.055228 rpy=0 0 0; parent base_link -> container_link
- joint wheel_left_joint: origin xyz=0 0.043423 0.028 rpy=0 0 0 -> xyz=0 0.056 0.028 rpy=0 0 0; parent base_link -> body_link
- joint wheel_right_joint: origin xyz=0 -0.043423 0.028 rpy=0 0 0 -> xyz=0 -0.056 0.028 rpy=0 0 0; parent base_link -> body_link

Commit message: Update models/etrobo_spike/model.sdf

File: urdf/etrobo_spike.urdf (robot description, URDF)
Before this commit: robot etrobo_spike, 8 links, 7 joints
Links:
- link head_link: geometry collision box size=0.080 0.072 0.064; visual box size=0.080 0.072 0.064
